File: hardware/sd_locker.sch (KiCad schematic (older format))
At the start: 17 parts, among them J1 USB_OTG, J2 3V3, J3 5V, J4 SD_Card, Q1 Q_PMOS_GSD, SW1 SW_Push, U1 AP1117-33, U2 ATTINY85-20SU

Commit message: Unverified - fixing the SD locker PCB layout so that airwires are not needed for SD slot connection, adding proper CD wire, adding 0R resistor for easier "battery-powered SD locker" modding
Parts:
- added R5: 0, Resistors_SMD:R_0603_HandSoldering, symbol sd_locker-rescue:R_Small
- C1, C2, C3, C4: symbol C_Small -> sd_locker-rescue:C_Small
- D1: symbol LED -> sd_locker-rescue:LED
- J1: symbol USB_OTG -> sd_locker-rescue:USB_OTG
- J2: symbol Conn_01x02 -> sd_locker-rescue:Conn_01x02
- J3: value 5V -> VIN; symbol Conn_01x02 -> sd_locker-rescue:Conn_01x02
- J4: symbol SD_Card -> sd_locker-rescue:SD_Card
- Q1: symbol Q_PMOS_GSD -> sd_locker-rescue:Q_PMOS_GSD
- R1, R2, R3, R4: symbol R_Small -> sd_locker-rescue:R_Small
- SW1: symbol SW_Push -> sd_locker-rescue:SW_Push
- U1: symbol AP1117-33 -> sd_locker-rescue:AP1117-33
- U2: symbol ATTINY85-20SU -> sd_locker-rescue:ATTINY85-20SU
Connections:
- net +5V: no longer J3.2 (Pin_2)
- net VBUS: now also J3.2 (Pin_2), R5.1; no longer J1.1 (VBUS)
- new net: J1.1 (VBUS), R5.2
Changed lines of the file:
@@
-EESchema Schematic File Version 2
-LIBS:power
-LIBS:device
-LIBS:switches
-LIBS:relays
-LIBS:motors
-LIBS:transistors
-LIBS:conn
-LIBS:linear
-LIBS:regul
-LIBS:74xx
-LIBS:cmos4000
-LIBS:adc-dac
-LIBS:memory
-LIBS:xilinx
-LIBS:microcontrollers
-LIBS:dsp
-LIBS:microchip
-LIBS:analog_switches
-LIBS:motorola
-LIBS:texas
-LIBS:intel
-LIBS:audio
-LIBS:interface
-LIBS:digital-audio
-LIBS:philips
-LIBS:display
-LIBS:cypress
-LIBS:siliconi
-LIBS:opto
-LIBS:atmel
-LIBS:contrib
-LIBS:valves
+EESchema Schematic File Version 4
 LIBS:sd_locker-cache
-EELAYER 25 0
+EELAYER 26 0
 EELAYER END
 $Descr A4 11693 8268
@@
 $EndDescr
 $Comp
-L ATTINY85-20SU U2
+L sd_locker-rescue:ATTINY85-20SU U2
 U 1 1 5BA87E84
 P 4550 3750
@@
 $EndComp
 $Comp
-L +3.3V #PWR01
+L power:+3.3V #PWR01
 U 1 1 5BA87EDA
 P 5900 3500
@@
 $EndComp
 $Comp
-L GND #PWR02
+L power:GND #PWR02
 U 1 1 5BA87EF0
 P 5900 4000
@@
 $EndComp
 $Comp
-L R_Small R1
+L sd_locker-rescue:R_Small R1
 U 1 1 5BA87F13
 P 3100 4200
@@
 $EndComp
 $Comp
-L +3.3V #PWR03
+L power:+3.3V #PWR03
 U 1 1 5BA87F40
 P 3100 4400
@@
 LEDSW
 $Comp
-L LED D1
+L sd_locker-rescue:LED D1
 U 1 1 5BA87FE0
 P 3800 2100
@@
 $EndComp
 $Comp
-L R_Small R3
+L sd_locker-rescue:R_Small R3
 U 1 1 5BA8801D
 P 4200 2100
@@
 $EndComp
 $Comp
-L +3.3V #PWR04
+L power:+3.3V #PWR04
 U 1 1 5BA88084
 P 3500 2100
@@
 	4300 2100 4400 2100
 $Comp
-L R_Small R2
+L sd_locker-rescue:R_Small R2
 U 1 1 5BA880F6
 P 3800 2450
@@
 MOSI
 $Comp
-L SD_Card J4
+L sd_locker-rescue:SD_Card J4
 U 1 1 5BA881DD
 P 7300 2300
@@
 $EndComp
 $Comp
-L +3.3V #PWR05
+L power:+3.3V #PWR05
 U 1 1 5BA88278
 P 6400 2300
@@
 $EndComp
 $Comp
-L GND #PWR06
+L power:GND #PWR06
 U 1 1 5BA882AD
 P 6400 2200
@@
 $EndComp
 $Comp
-L GND #PWR07
+L power:GND #PWR07
 U 1 1 5BA882ED
 P 6400 2500
@@
 NoConn ~ 6400 2700
 $Comp
-L GND #PWR08
+L power:GND #PWR08
 U 1 1 5BA883BF
 P 8200 2500
@@
 $EndComp
 $Comp
-L GND #PWR09
+L power:GND #PWR09
 U 1 1 5BA883DC
 P 8200 2400
@@
 NoConn ~ 8200 2200
 $Comp
-L USB_OTG J1
+L sd_locker-rescue:USB_OTG J1
 U 1 1 5BA8841C
 P 1900 2800
@@
 $EndComp
 $Comp
-L +5V #PWR010
+L power:+5V #PWR010
 U 1 1 5BA884A2
 P 5250 1200
@@
 Wire Wire Line
 	2200 2600 2250 2600
-Wire Wire Line
-	2250 2600 2250 2550
-$Comp
-L GND #PWR011
+$Comp
+L power:GND #PWR011
 U 1 1 5BA884FC
 P 1800 3200
@@
 $EndComp
 $Comp
-L GND #PWR012
+L power:GND #PWR012
 U 1 1 5BA8853F
 P 1900 3350
@@
 NoConn ~ 2200 3000
 $Comp
-L C_Small C3
+L sd_locker-rescue:C_Small C3
 U 1 1 5BA885F6
 P 5900 3750
@@
 Connection ~ 5900 3500
 $Comp
-L AP1117-33 U1
+L sd_locker-rescue:AP1117-33 U1
 U 1 1 5BA88706
 P 3900 1250
@@
 $EndComp
 $Comp
-L +3.3V #PWR013
+L power:+3.3V #PWR013
 U 1 1 5BA8877E
 P 4200 1250
@@
 $EndComp
 $Comp
-L +5V #PWR014
+L power:+5V #PWR014
 U 1 1 5BA887A4
 P 3600 1250
@@
 $EndComp
 $Comp
-L GND #PWR015
+L power:GND #PWR015
 U 1 1 5BA88814
 P 3900 1550
@@
 $EndComp
 $Comp
-L C_Small C2
+L sd_locker-rescue:C_Small C2
 U 1 1 5BA88833
 P 4600 1400
@@
 $EndComp
 $Comp
-L +3.3V #PWR016
+L power:+3.3V #PWR016
 U 1 1 5BA8889E
 P 4600 1300
@@
 $EndComp
 $Comp
-L GND #PWR017
+L power:GND #PWR017
 U 1 1 5BA888C7
 P 4600 1500
@@
 $EndComp
 $Comp
-L C_Small C1
+L sd_locker-rescue:C_Small C1
 U 1 1 5BA888F0
 P 3050 1400
@@
 $EndComp
 $Comp
-L GND #PWR018
+L power:GND #PWR018
 U 1 1 5BA8899E
 P 3050 1500
@@
 $EndComp
 $Comp
-L +5V #PWR019
+L power:+5V #PWR019
 U 1 1 5BA889C1
 P 3050 1300
@@
 TODO:\n\n- Add MOSFET to switch from CARD_DETECT\n- Add button\n- Add SD footprint
 $Comp
-L SW_Push SW1
+L sd_locker-rescue:SW_Push SW1
 U 1 1 5BCD1502
 P 4100 2450
@@
 $EndComp
 $Comp
-L GND #PWR020
+L power:GND #PWR020
 U 1 1 5BCD15AD
 P 4300 2450
@@
 $EndComp
 $Comp
-L Q_PMOS_GSD Q1
+L sd_locker-rescue:Q_PMOS_GSD Q1
 U 1 1 5BCD173E
 P 5700 1300
@@
 CD
 $Comp
-L VBUS #PWR021
+L power:VBUS #PWR021
 U 1 1 5BCD1988
-P 2250 2550
-F 0 "#PWR021" H 2250 2400 50  0001 C CNN
-F 1 "VBUS" H 2250 2700 50  0000 C CNN
-F 2 "" H 2250 2550 50  0001 C CNN
-F 3 "" H 2250 2550 50  0001 C CNN
-	1    2250 2550
-	1    0    0    -1
-$EndComp
-$Comp
-L VBUS #PWR022
+P 2550 2550
+F 0 "#PWR021" H 2550 2400 50  0001 C CNN
+F 1 "VBUS" H 2550 2700 50  0000 C CNN
+F 2 "" H 2550 2550 50  0001 C CNN
+F 3 "" H 2550 2550 50  0001 C CNN
+	1    2550 2550
+	1    0    0    -1
+$EndComp
+$Comp
+L power:VBUS #PWR022
 U 1 1 5BCD1A23
 P 6050 1150
@@
 $EndComp
 $Comp
-L R_Small R4
+L sd_locker-rescue:R_Small R4
 U 1 1 5BCD1ACA
 P 6000 1450
@@
 $EndComp
 Wire Wire Line
-	5900 1200 6050 1200
+	5900 1200 6000 1200
 Wire Wire Line
 	6050 1200 6050 1150
@@
 	5700 1500 5700 1600
 Wire Wire Line
-	5500 1600 6000 1600
+	5500 1600 5700 1600
 Wire Wire Line
 	6000 1600 6000 1550
@@
 	5250 1200 5500 1200
 $Comp
-L Conn_01x02 J2
+L sd_locker-rescue:Conn_01x02 J2
 U 1 1 5BCD1E4F
 P 2050 1200
@@
 $EndComp
 $Comp
-L +3.3V #PWR023
+L power:+3.3V #PWR023
 U 1 1 5BCD1F2A
 P 2250 1100
@@
 $EndComp
 $Comp
-L GND #PWR024
+L power:GND #PWR024
 U 1 1 5BCD1F62
 P 2250 1200
@@
 $EndComp
 $Comp
-L Conn_01x02 J3
+L sd_locker-rescue:Conn_01x02 J3
 U 1 1 5BCD1F9A
 P 2050 1600
 F 0 "J3" H 2050 1700 50  0000 C CNN
-F 1 "5V" H 2050 1400 50  0000 C CNN
+F 1 "VIN" H 2050 1400 50  0000 C CNN
 F 2 "Pin_Headers:Pin_Header_Straight_1x02_Pitch2.54mm" H 2050 1600 50  0001 C CNN
 F 3 "" H 2050 1600 50  0001 C CNN
@@
 $EndComp
 $Comp
-L +5V #PWR025
-U 1 1 5BCD2030
-P 2250 1500
-F 0 "#PWR025" H 2250 1350 50  0001 C CNN
-F 1 "+5V" V 2250 1700 50  0000 C CNN
-F 2 "" H 2250 1500 50  0001 C CNN
-F 3 "" H 2250 1500 50  0001 C CNN
-	1    2250 1500
-	0    1    1    0
-$EndComp
-$Comp
-L GND #PWR026
+L power:GND #PWR026
 U 1 1 5BCD20B5
 P 2250 1600
@@
 $EndComp
 $Comp
-L C_Small C4
+L sd_locker-rescue:C_Small C4
 U 1 1 5BCD1967
 P 4950 1400
@@
 $EndComp
 $Comp
-L GND #PWR027
+L power:GND #PWR027
 U 1 1 5BCD19B0
 P 4950 1500
@@
 $EndComp
 $Comp
-L +3.3V #PWR028
+L power:+3.3V #PWR028
 U 1 1 5BCD19EE
 P 4950 1300
@@
 	1    0    0    -1
 $EndComp
+Wire Wire Line
+	6000 1200 6050 1200
+Wire Wire Line
+	5700 1600 6000 1600
+$Comp
+L power:VBUS #PWR0101
+U 1 1 5DBE9517
+P 2250 1500
+F 0 "#PWR0101" H 2250 1350 50  0001 C CNN
+F 1 "VBUS" V 2250 1700 50  0000 C CNN
+F 2 "" H 2250 1500 50  0001 C CNN
+F 3 "" H 2250 1500 50  0001 C CNN
+	1    2250 1500
+	0    1    1    0
+$EndComp
+$Comp
+L sd_locker-rescue:R_Small R5
+U 1 1 5DBE97F2
+P 2350 2600
+F 0 "R5" V 2350 2550 50  0000 L CNN
+F 1 "0" V 2250 2550 50  0000 L CNN
+F 2 "Resistors_SMD:R_0603_HandSoldering" H 2350 2600 50  0001 C CNN
+F 3 "" H 2350 2600 50  0001 C CNN
+	1    2350 2600
+	0    1    1    0
+$EndComp
+Wire Wire Line
+	2450 2600 2550 2600
+Wire Wire Line
+	2550 2600 2550 2550
 $EndSCHEMATC

Commit message: Latest hardware version (v2) added
Parts:
- added C5: 100nF, sd_locker:C_0805_100nF_HandSoldering, symbol sd_locker-rescue:C_Small
- added FID1: Fiducial, Fiducial:Fiducial_1.5mm_Mask3mm, symbol Mechanical:Fiducial
- added J5: Micro_SD_Card_Det, sd_locker:microSD-Receptacle-SelfEject, symbol Connector:Micro_SD_Card_Det
Connections:
- net +3V3: now also C5.1, J5.4 (VDD)
- net CD: now also J5.10 (DET_A)
- net CS: now also J5.2 (DAT3/CD)
- net GND: now also C5.2, J5.11 (SHIELD), J5.6 (VSS)
- net MISO: now also J5.7 (DAT0)
- net MOSI: now also J5.3 (CMD)
- net SCK: now also J5.5 (CLK)
- no-connect marks 6 -> 9
Other:
- note removed: "TODO:\n\n- Add MOSFET to switch from CARD_DETECT\n- Add button\n- Add SD footprint"
- moved on the sheet: Q1, R4
Changed lines of the file:
@@
 EESchema Schematic File Version 4
 LIBS:sd_locker-cache
-EELAYER 26 0
+EELAYER 29 0
 EELAYER END
 $Descr A4 11693 8268
@@
 L power:+5V #PWR010
 U 1 1 5BA884A2
-P 5250 1200
-F 0 "#PWR010" H 5250 1050 50  0001 C CNN
-F 1 "+5V" H 5250 1340 50  0000 C CNN
-F 2 "" H 5250 1200 50  0001 C CNN
-F 3 "" H 5250 1200 50  0001 C CNN
-	1    5250 1200
+P 5600 1200
+F 0 "#PWR010" H 5600 1050 50  0001 C CNN
+F 1 "+5V" H 5600 1340 50  0000 C CNN
+F 2 "" H 5600 1200 50  0001 C CNN
+F 3 "" H 5600 1200 50  0001 C CNN
+	1    5600 1200
 	1    0    0    -1
 $EndComp
@@
 	1    0    0    -1
 $EndComp
-Text Notes 3300 3250 0    60   ~ 0
-TODO:\n\n- Add MOSFET to switch from CARD_DETECT\n- Add button\n- Add SD footprint
 $Comp
 L sd_locker-rescue:SW_Push SW1
@@
 L sd_locker-rescue:Q_PMOS_GSD Q1
 U 1 1 5BCD173E
-P 5700 1300
-F 0 "Q1" H 5900 1350 50  0000 L CNN
-F 1 "Q_PMOS_GSD" V 6050 1100 50  0000 L CNN
-F 2 "sd_locker:IRLML6401-SOT-23_Handsoldering" H 5900 1400 50  0001 C CNN
-F 3 "" H 5700 1300 50  0001 C CNN
-	1    5700 1300
+P 6050 1300
+F 0 "Q1" H 6250 1350 50  0000 L CNN
+F 1 "Q_PMOS_GSD" V 6400 1100 50  0000 L CNN
+F 2 "sd_locker:IRLML6401-SOT-23_Handsoldering" H 6250 1400 50  0001 C CNN
+F 3 "" H 6050 1300 50  0001 C CNN
+	1    6050 1300
 	0    -1   -1   0
 $EndComp
 Text GLabel 8200 2100 2    60   Input ~ 0
 CD
-Text GLabel 5500 1600 0    60   Input ~ 0
+Text GLabel 5850 1600 0    60   Input ~ 0
 CD
 $Comp
@@
 L power:VBUS #PWR022
 U 1 1 5BCD1A23
-P 6050 1150
-F 0 "#PWR022" H 6050 1000 50  0001 C CNN
-F 1 "VBUS" H 6050 1300 50  0000 C CNN
-F 2 "" H 6050 1150 50  0001 C CNN
-F 3 "" H 6050 1150 50  0001 C CNN
-	1    6050 1150
+P 6400 1150
+F 0 "#PWR022" H 6400 1000 50  0001 C CNN
+F 1 "VBUS" H 6400 1300 50  0000 C CNN
+F 2 "" H 6400 1150 50  0001 C CNN
+F 3 "" H 6400 1150 50  0001 C CNN
+	1    6400 1150
 	1    0    0    -1
 $EndComp
@@
 L sd_locker-rescue:R_Small R4
 U 1 1 5BCD1ACA
-P 6000 1450
-F 0 "R4" V 6000 1400 50  0000 L CNN
-F 1 "10K" V 5900 1400 50  0000 L CNN
-F 2 "sd_locker:R_0805_10K_HandSoldering" H 6000 1450 50  0001 C CNN
-F 3 "" H 6000 1450 50  0001 C CNN
-	1    6000 1450
+P 6350 1450
+F 0 "R4" V 6350 1400 50  0000 L CNN
+F 1 "10K" V 6250 1400 50  0000 L CNN
+F 2 "sd_locker:R_0805_10K_HandSoldering" H 6350 1450 50  0001 C CNN
+F 3 "" H 6350 1450 50  0001 C CNN
+	1    6350 1450
 	-1   0    0    1
 $EndComp
 Wire Wire Line
-	5900 1200 6000 1200
-Wire Wire Line
-	6050 1200 6050 1150
-Wire Wire Line
-	6000 1200 6000 1350
-Connection ~ 6000 1200
-Wire Wire Line
-	5700 1500 5700 1600
-Wire Wire Line
-	5500 1600 5700 1600
-Wire Wire Line
-	6000 1600 6000 1550
-Connection ~ 5700 1600
-Wire Wire Line
-	5250 1200 5500 1200
+	6250 1200 6350 1200
+Wire Wire Line
+	6400 1200 6400 1150
+Wire Wire Line
+	6350 1200 6350 1350
+Connection ~ 6350 1200
+Wire Wire Line
+	6050 1500 6050 1600
+Wire Wire Line
+	5850 1600 6050 1600
+Wire Wire Line
+	6350 1600 6350 1550
+Connection ~ 6050 1600
+Wire Wire Line
+	5600 1200 5850 1200
 $Comp
 L sd_locker-rescue:Conn_01x02 J2
@@
 $EndComp
 Wire Wire Line
-	6000 1200 6050 1200
-Wire Wire Line
-	5700 1600 6000 1600
+	6350 1200 6400 1200
+Wire Wire Line
+	6050 1600 6350 1600
 $Comp
 L power:VBUS #PWR0101
@@
 Wire Wire Line
 	2550 2600 2550 2550
+$Comp
+L Mechanical:Fiducial FID1
+U 1 1 5DCCB5E6
+P 1150 1000
+F 0 "FID1" H 1235 1046 50  0000 L CNN
+F 1 "Fiducial" H 1235 955 50  0000 L CNN
+F 2 "Fiducial:Fiducial_1.5mm_Mask3mm" H 1150 1000 50  0001 C CNN
+F 3 "~" H 1150 1000 50  0001 C CNN
+	1    1150 1000
+	1    0    0    -1
+$EndComp
+Text GLabel 7000 4350 0    60   Input ~ 0
+CD
+$Comp
+L Connector:Micro_SD_Card_Det J5
+U 1 1 5DCD5886
+P 7900 3950
+F 0 "J5" H 7850 4767 50  0000 C CNN
+F 1 "Micro_SD_Card_Det" H 7850 4676 50  0000 C CNN
+F 2 "sd_locker:microSD-Receptacle-SelfEject" H 9950 4650 50  0001 C CNN
+F 3 "https://www.hirose.com/product/en/download_file/key_name/DM3/category/Catalog/doc_file_id/49662/?file_category_id=4&item_id=195&is_series=1" H 7900 4050 50  0001 C CNN
+	1    7900 3950
+	1    0    0    -1
+$EndComp
+NoConn ~ 7000 4450
+Text GLabel 7000 4150 0    60   Input ~ 0
+MISO
+$Comp
+L power:GND #PWR0102
+U 1 1 5DCD816F
+P 7000 4050
+F 0 "#PWR0102" H 7000 3800 50  0001 C CNN
+F 1 "GND" V 7000 3850 50  0000 C CNN
+F 2 "" H 7000 4050 50  0001 C CNN
+F 3 "" H 7000 4050 50  0001 C CNN
+	1    7000 4050
+	0    1    1    0
+$EndComp
+Text GLabel 7000 3950 0    60   Input ~ 0
+SCK
+$Comp
+L power:+3.3V #PWR0103
+U 1 1 5DCD85F9
+P 7000 3850
+F 0 "#PWR0103" H 7000 3700 50  0001 C CNN
+F 1 "+3.3V" V 7000 4100 50  0000 C CNN
+F 2 "" H 7000 3850 50  0001 C CNN
+F 3 "" H 7000 3850 50  0001 C CNN
+	1    7000 3850
+	0    -1   -1   0
+$EndComp
+Text GLabel 7000 3750 0    60   Input ~ 0
+MOSI
+Text GLabel 7000 3650 0    60   Input ~ 0
+CS
+NoConn ~ 7000 4250
+NoConn ~ 7000 3550
+$Comp
+L power:GND #PWR0104
+U 1 1 5DCD998C
+P 8700 4450
+F 0 "#PWR0104" H 8700 4200 50  0001 C CNN
+F 1 "GND" V 8700 4250 50  0000 C CNN
+F 2 "" H 8700 4450 50  0001 C CNN
+F 3 "" H 8700 4450 50  0001 C CNN
+	1    8700 4450
+	0    -1   -1   0
+$EndComp
+$Comp
+L sd_locker-rescue:C_Small C5
+U 1 1 5DCF1768
+P 5300 1400
+F 0 "C5" H 5310 1470 50  0000 L CNN
+F 1 "100nF" H 5310 1320 50  0000 L CNN
+F 2 "sd_locker:C_0805_100nF_HandSoldering" H 5300 1400 50  0001 C CNN
+F 3 "" H 5300 1400 50  0001 C CNN
+	1    5300 1400
+	1    0    0    -1
+$EndComp
+$Comp
+L power:+3.3V #PWR0105
+U 1 1 5DCF1772
+P 5300 1300
+F 0 "#PWR0105" H 5300 1150 50  0001 C CNN
+F 1 "+3.3V" H 5300 1440 50  0000 C CNN
+F 2 "" H 5300 1300 50  0001 C CNN
+F 3 "" H 5300 1300 50  0001 C CNN
+	1    5300 1300
+	1    0    0    -1
+$EndComp
+$Comp
+L power:GND #PWR0106
+U 1 1 5DCF177C
+P 5300 1500
+F 0 "#PWR0106" H 5300 1250 50  0001 C CNN
+F 1 "GND" H 5300 1350 50  0000 C CNN
+F 2 "" H 5300 1500 50  0001 C CNN
+F 3 "" H 5300 1500 50  0001 C CNN
+	1    5300 1500
+	1    0    0    -1
+$EndComp
 $EndSCHEMATC

Commit message: Adding a fiducial on the bottom layer
Parts:
- added FID2: Fiducial, Fiducial:Fiducial_1.5mm_Mask3mm, symbol Mechanical:Fiducial
Changed lines of the file:
@@
+	1    0    0    -1
+$EndComp
+$Comp
+L Mechanical:Fiducial FID2
+U 1 1 5DD45667
+P 1150 1200
+F 0 "FID2" H 1235 1246 50  0000 L CNN
+F 1 "Fiducial" H 1235 1155 50  0000 L CNN
+F 2 "Fiducial:Fiducial_1.5mm_Mask3mm" H 1150 1200 50  0001 C CNN
+F 3 "~" H 1150 1200 50  0001 C CNN
+	1    1150 1200
 	1    0    0    -1
 $EndComp

Commit message: Latest hardware revision, v3, wasn't uplaoded for a long time - fixed
Parts:
- added R6: 0, Resistor_SMD:R_0603_1608Metric_Pad1.05x0.95mm_HandSolder, symbol sd_locker-rescue:R_Small
- R5: footprint Resistors_SMD:R_0603_HandSoldering -> Resistor_SMD:R_0603_1608Metric_Pad1.05x0.95mm_HandSolder
Connections:
- net RST: now reaches R1.2, U2.1 (PB5(~RESET~/dW/ADC0/PCINT5))
- net RST: now also R6.2
- net at J4.8 (DAT1): now also R6.1
- no-connect marks 9 -> 8
Other:
- note added: "RST is connected to DAT1 purely to allow\nreprogramming the ATTiny through\nthe large SD card socket."
- note added: "power management - powers the circuit\nwhen CD is pulled to GND through one\nof the sockets"
Changed lines of the file:
@@
 EESchema Schematic File Version 4
-LIBS:sd_locker-cache
-EELAYER 29 0
+EELAYER 30 0
 EELAYER END
 $Descr A4 11693 8268
@@
 CS
 NoConn ~ 6400 1900
-NoConn ~ 6400 2700
 $Comp
 L power:GND #PWR08
@@
 F 0 "R5" V 2350 2550 50  0000 L CNN
 F 1 "0" V 2250 2550 50  0000 L CNN
-F 2 "Resistors_SMD:R_0603_HandSoldering" H 2350 2600 50  0001 C CNN
+F 2 "Resistor_SMD:R_0603_1608Metric_Pad1.05x0.95mm_HandSolder" H 2350 2600 50  0001 C CNN
 F 3 "" H 2350 2600 50  0001 C CNN
 	1    2350 2600
@@
 	1    0    0    -1
 $EndComp
+Text GLabel 2900 4000 0    50   Input ~ 0
+RST
+Wire Wire Line
+	2900 4000 3100 4000
+Connection ~ 3100 4000
+$Comp
+L sd_locker-rescue:R_Small R6
+U 1 1 5E1E87AC
+P 6000 2700
+F 0 "R6" V 6000 2650 50  0000 L CNN
+F 1 "0" V 5900 2650 50  0000 L CNN
+F 2 "Resistor_SMD:R_0603_1608Metric_Pad1.05x0.95mm_HandSolder" H 6000 2700 50  0001 C CNN
+F 3 "" H 6000 2700 50  0001 C CNN
+	1    6000 2700
+	0    1    1    0
+$EndComp
+Text GLabel 5900 2700 0    50   Input ~ 0
+RST
+Wire Wire Line
+	6100 2700 6400 2700
+Text Notes 4900 3100 0    50   ~ 0
+RST is connected to DAT1 purely to allow\nreprogramming the ATTiny through\nthe large SD card socket.
+Text Notes 6550 1350 0    50   ~ 0
+power management - powers the circuit\nwhen CD is pulled to GND through one\nof the sockets
 $EndSCHEMATC
